Commit message: created new control file

File: description/gazebo_control.xacro (robot description, xacro)
@@ -1,21 +1,21 @@
 <?xml version="1.0"?>
-<robot xmlns:xacro="http://www.ros.org/wiki/xacro"  name="robot">
+<robot xmlns:xacro="http://www.ros.org/wiki/xacro">
     <gazebo>
-        <plugin name="diff_drive" filename="libagazebo_ros_diff_drive.so">
-        <!--wheel information-->
-        <left_joint>left_wheel_joint</left_joint>
-        <right_joint>right_wheel_joint</right_joint>
-        <wheel_seperation>0.35</wheel_seperation>
-        <wheel_diameter>0.1</wheel_diameter>
-        <!--limits-->
-        <max_wheel_torque>200</max_wheel_torque>
-        <max_wheel_acceleration>10.0</max_wheel_acceleration>
-        <!--Output-->
-        <odometry_frame>odom</odometry_frame>
-        <robot_base_frame>base_link</robot_base_frame>
-        <publish_odom>true</publish_odom>
-        <publish_odom_tf>true</publish_odom_tf>
-        <publish_wheel_tf>true</publish_wheel_tf>
-    </plugin>
-</gazebo>
+        <plugin name="diff_drive" filename="libgazebo_ros_diff_drive.so">
+            <!-- Wheel Information -->
+            <left_joint>left_wheel_joint</left_joint>
+            <right_joint>right_wheel_joint</right_joint>
+            <wheel_separation>0.35</wheel_separation>
+            <wheel_diameter>0.1</wheel_diameter>
+            <!-- Limits -->
+            <max_wheel_torque>200</max_wheel_torque>
+            <max_wheel_acceleration>10.0</max_wheel_acceleration>
+            <!-- Output -->
+            <odometry_frame>odom</odometry_frame>
+            <robot_base_frame>base_link</robot_base_frame>
+            <publish_odom>true</publish_odom>
+            <publish_odom_tf>true</publish_odom_tf>
+            <publish_wheel_tf>true</publish_wheel_tf>
+        </plugin>
+    </gazebo>
 </robot>

File: description/robot_core.xacro (robot description, xacro)
@@ -5,17 +5,17 @@
         <color rgba="1 1 1 1" />
     </material>
-           <material name="orange">
-        <color rgba="1 0.3 0.1 1" />
+    <material name="orange">
+        <color rgba="1 0.3 0.1 1"/>
     </material>
-        <material name="blue">
-        <color rgba="0.2 0.2 1 1" />
+    <material name="blue">
+        <color rgba="0.2 0.2 1 1"/>
     </material>
-        <material name="black">
-        <color rgba="0 0 0 1" />
+    <material name="black">
+        <color rgba="0 0 0 1"/>
     </material>
-    <!--BASE LINK -->
+    <!-- BASE LINK -->
     <link name="base_link">
     </link>
-    <!--CHASSIS LINK-->
+    <!-- CHASSIS LINK -->
     <joint name="chassis_joint" type="fixed">
         <parent link="base_link"/>
@@ -25,29 +25,29 @@
     <link name="chassis">
         <visual>
-            <origin xyz="0.15 0 0.075" />
+            <origin xyz="0.15 0 0.075"/>
             <geometry>
-                <box size="0.3 0.3 0.15" />
+                <box size="0.3 0.3 0.15"/>
             </geometry>
-            <material name="white" />
+            <material name="white"/>
         </visual>
-             <collision>
-            <origin xyz="0.15 0 0.075" />
+        <collision>
+            <origin xyz="0.15 0 0.075"/>
             <geometry>
-                <box size="0.3 0.3 0.15" />
+                <box size="0.3 0.3 0.15"/>
             </geometry>
         </collision>
         <xacro:inertial_box mass="0.5" x="0.3" y="0.3" z="0.15">
-            <origin xyz="0.15 0.15 0.075" rpy="0 0 0"/>
+            <origin xyz="0.15 0 0.075" rpy="0 0 0"/>
         </xacro:inertial_box>
-     </link>
+    </link>
     <gazebo reference="chassis">
-    <material>Gazebo/White</material>
+        <material>Gazebo/White</material>
     </gazebo>
-    <!--LEFT WHEEL LINK-->
+    <!-- LEFT WHEEL LINK -->
     <joint name="left_wheel_joint" type="continuous">
         <parent link="base_link"/>
         <child link="left_wheel"/>
         <origin xyz="0 0.175 0" rpy="-${pi/2} 0 0" />
-        <axis xyz= "0 0 1"/>
+        <axis xyz="0 0 1"/>
     </joint>
     <link name="left_wheel">
@@ -56,5 +56,5 @@
                 <cylinder radius="0.05" length="0.04"/>
             </geometry>
-            <material name="blue" />
+            <material name="blue"/>
         </visual>
         <collision>
@@ -68,12 +68,12 @@
     </link>
     <gazebo reference="left_wheel">
-    <material>Gazebo/Blue</material>
+        <material>Gazebo/Blue</material>
     </gazebo>
- <!--RIGHT WHEEL LINK-->
+    <!-- RIGHT WHEEL LINK -->
     <joint name="right_wheel_joint" type="continuous">
-        <parent link="base_link" />
-        <child link="right_wheel" />
-        <origin xyz="0 -0.175 0" rpy="${pi/2} 0 0"/>
-        <axis xyz= "0 0 -1"/>
+        <parent link="base_link"/>
+        <child link="right_wheel"/>
+        <origin xyz="0 -0.175 0" rpy="${pi/2} 0 0" />
+        <axis xyz="0 0 -1"/>
     </joint>
     <link name="right_wheel">
@@ -84,18 +84,17 @@
             <material name="blue"/>
         </visual>
-                <collision>
+        <collision>
             <geometry>
                 <cylinder radius="0.05" length="0.04"/>
             </geometry>
-            <material name="blue"/>
         </collision>
-                <xacro:inertial_cylinder mass="0.1" length="0.04" radius="0.05">
+        <xacro:inertial_cylinder mass="0.1" length="0.04" radius="0.05">
             <origin xyz="0 0 0" rpy="0 0 0"/>
         </xacro:inertial_cylinder>
     </link>
     <gazebo reference="right_wheel">
-    <material>Gazebo/Blue</material>
+        <material>Gazebo/Blue</material>
     </gazebo>
-    <!--CASTER WHEEL LINK -->
+    <!-- CASTER WHEEL LINK -->
     <joint name="caster_wheel_joint" type="fixed">
         <parent link="chassis"/>
@@ -110,5 +109,5 @@
             <material name="black"/>
         </visual>
-                <collision>
+        <collision>
             <geometry>
                 <sphere radius="0.05"/>
@@ -120,7 +119,7 @@
     </link>
     <gazebo reference="caster_wheel">
-    <material>Gazebo/Black</material>
-    <mu1 value="0.001" />
-    <mu2 value="0.001" />
+        <material>Gazebo/Black</material>
+        <mu1 value="0.001"/>
+        <mu2 value="0.001"/>
     </gazebo>
 </robot>
